File: design_pcb/copter.brd (EAGLE design)
At the start: 35.6 x 35.6 mm, 52 parts, among them U1 ATMEGA328P-AU, U10 INA169, U2 ITG-3200, U3 ADXL345, U5 HC_05, U6 IRF9362PBF, U7 IRF9362PBF, U8 HMC5883LSMD, U9 3.3V, X1 05-JST-B5B-XH-A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

Commit message: merge from other repository
Parts:
- removed X1: 05-JST-B5B-XH-A, bt_con-jst-xh:B5B-XH
- added J1: USB-MINIB-5PIN, SparkFun-Connectors:USB-MINIB
- added R2, R3: 1k, resistor:R0402
- added U$1: CH340G, usb-serial:SOIC16
- added U$2: CSTCV, murata-cstcc-cstce-cstcr-cstcv-resonators:CSTCV
- moved VIN_PAD 36.6 mm to (25.4, 1.91)
- moved GND_PAD 36.6 mm to (27.3, 1.91)
- moved C2_5V1 31.5 mm to (25.4, 6.35), flipped to the bottom, turned to 180 degrees
- moved C1_5V1 30.7 mm to (25.9, 4.55), flipped to the bottom, turned to 180 degrees
- moved R_SHUNT 25.7 mm to (13.3, 10.2), flipped to the bottom
- moved MTR4_2 23.8 mm to (5.71, 3.81)
- moved MTR3_2 23.8 mm to (5.71, 31.8)
- moved MTR1_1 21.9 mm to (29.8, 3.81)
- moved MTR2_1 21.9 mm to (29.8, 31.8)
- moved MTR1_2 21.7 mm to (31.8, 5.71)
- moved MTR2_2 21.7 mm to (31.8, 29.8)
- moved MTR3_1 19.8 mm to (3.81, 29.8)
- moved MTR4_1 19.8 mm to (3.81, 5.71)
- moved C1_3V1 15.9 mm to (1.91, 13.3)
- moved U9 15.5 mm to (2.29, 10.2)
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Connections:
- new net D+: J1.D+, U$1.5
- new net D-: J1.D-, U$1.6
- new net N$1: R2.2, U$1.2
- new net N$16: U$1.7, U$2.IN
- new net N$4: R3.2, U$1.3
- new net N$9: U$1.8, U$2.OUT
- net +5V: now also J1.VBUS, U$1.16; no longer X1.P$5
- net D0/RX: now also R3.1; no longer X1.P$2
- net D1/TX: now also R2.1; no longer X1.P$3
- net DTR: now also U$1.13; no longer X1.P$4
- net GND: now also J1.GND, U$1.1, U$2.GND; no longer X1.P$1
