File: design_pcb/copter.sch (EAGLE design)
At the start: 52 parts, among them U1 ATMEGA328P-AU, U10 INA169, U2 ITG-3200, U3 ADXL345, U5 HC_05, U6 IRF9362PBF, U7 IRF9362PBF, U8 HMC5883LSMD, U9 3.3V, X1 05-JST-B5B-XH-A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

Commit message: merge from other repository
Parts:
- removed X1: 05-JST-B5B-XH-A, bt_con-jst-xh:05-JST-B5B-XH-A
- added J1: USB-MINIB-5PIN, SparkFun-Connectors:USB-MINIB-5PIN
- added R2, R3: 1k, resistor:R-EU_R0402
- added U$1: CH340G, usb-serial:CH340G
- added U$2: CSTCV, murata-cstcc-cstce-cstcr-cstcv-resonators:CSTCV
Connections:
- new net D+: J1.D+, U$1.D+
- new net D-: J1.D-, U$1.D-
- new net N$1: R2.2, U$1.TX
- new net N$16: U$1.XI, U$2.IN
- new net N$4: R3.2, U$1.RX
- new net N$9: U$1.XO, U$2.OUT
- net +5V: now also J1.VBUS, U$1.VCC; no longer X1-5.1
- net D0/RX: now also R3.1; no longer X1-2.1
- net D1/TX: now also R2.1; no longer X1-3.1
- net DTR: now also U$1.DTR; no longer X1-4.1
- net GND: now also J1.GND, U$1.GND, U$2.GND; no longer X1-1.1
Other:
- note removed: "SPI"
